File: PCB/CYOA_Ortho.kicad_pcb (KiCad board)
At the start: 2 copper layers, 229.2 x 95.5 mm, 149 parts, among them U1 ProMicro

Commit message: Layout done, routing started
Parts:
- added REF**: MountingHole_2.2mm_M2, MountingHole:MountingHole_2.2mm_M2, F.Cu at (226.8, 74.0)
- added REF**: MountingHole_2.2mm_M2, MountingHole:MountingHole_2.2mm_M2, F.Cu at (150.4, 112.2)
- added REF**: MountingHole_2.2mm_M2, MountingHole:MountingHole_2.2mm_M2, F.Cu at (226.8, 112.2)
- added REF**: MountingHole_2.2mm_M2, MountingHole:MountingHole_2.2mm_M2, F.Cu at (150.4, 74.0)
- added REF**: MountingHole_2.2mm_M2, MountingHole:MountingHole_2.2mm_M2, F.Cu at (112.2, 93.1)
- added REF**: MountingHole_2.2mm_M2, MountingHole:MountingHole_2.2mm_M2, F.Cu at (226.8, 54.9)
- added REF**: MountingHole_2.2mm_M2, MountingHole:MountingHole_2.2mm_M2, F.Cu at (188.6, 112.2)
- added REF**: MountingHole_2.2mm_M2, MountingHole:MountingHole_2.2mm_M2, F.Cu at (188.6, 74.0)
- added REF**: MountingHole_2.2mm_M2, MountingHole:MountingHole_2.2mm_M2, F.Cu at (74.0, 93.1)
- added REF**: MountingHole_2.2mm_M2, MountingHole:MountingHole_2.2mm_M2, F.Cu at (74.0, 112.2)
- added REF**: MountingHole_2.2mm_M2, MountingHole:MountingHole_2.2mm_M2, F.Cu at (150.4, 93.1)
- added REF**: MountingHole_2.2mm_M2, MountingHole:MountingHole_2.2mm_M2, F.Cu at (150.4, 54.9)
- added REF**: MountingHole_2.2mm_M2, MountingHole:MountingHole_2.2mm_M2, F.Cu at (112.2, 112.2)
- added REF**: MountingHole_2.2mm_M2, MountingHole:MountingHole_2.2mm_M2, F.Cu at (188.6, 54.9)
- added REF**: MountingHole_2.2mm_M2, MountingHole:MountingHole_2.2mm_M2, F.Cu at (226.8, 93.1)
- added REF**: MountingHole_2.2mm_M2, MountingHole:MountingHole_2.2mm_M2, F.Cu at (188.6, 93.1)
- added REF**: MountingHole_2.2mm_M2, MountingHole:MountingHole_2.2mm_M2, F.Cu at (112.2, 74.0)
- added REF**: MountingHole_2.2mm_M2, MountingHole:MountingHole_2.2mm_M2, F.Cu at (112.2, 54.9)
- moved U1 76.9 mm to (83.1, 59.9)
- moved REF** 76.3 mm to (169.4, 54.9)
- moved REF** 76.3 mm to (169.4, 74.0)
- moved D44 40.3 mm to (151.9, 83.6)
- moved D56 37.8 mm to (150.4, 129.4), turned to 0 degrees
- moved D7 35.5 mm to (168.0, 45.2)
- moved D19 35.5 mm to (168.0, 64.5)
- moved D55 19.5 mm to (131.3, 129.4), turned to 0 degrees
- moved D6 18.8 mm to (148.9, 45.2)
- moved D18 18.7 mm to (148.8, 64.5)
- moved D4 17.6 mm to (110.7, 45.5)
- moved D16 17.6 mm to (110.7, 64.5)
- moved D29 17.6 mm to (110.7, 83.6)
- moved D32 17.6 mm to (168.0, 83.3)
- moved D17 17.6 mm to (129.8, 64.5)
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Routing:
- net rowA: track 0.00 -> 154.7 mm
- net rowB: track 0.00 -> 143.1 mm
- net rowG: track 0.00 -> 141.9 mm
- net rowC: track 0.00 -> 140.3 mm
- net rowD: track 0.00 -> 138.4 mm
- net rowE: track 0.00 -> 119.1 mm
- net rowF: track 0.00 -> 118.3 mm
- net rowH: track 0.00 -> 59.6 mm
- net Net-(D44-Pad1): track 0.00 -> 49.1 mm
- net Net-(D3-Pad1): track 0.00 -> 32.1 mm
- net Net-(D43-Pad1): track 0.00 -> 31.1 mm
- net Net-(D42-Pad1): track 0.00 -> 29.2 mm
- net Net-(D54-Pad1): track 0.00 -> 21.5 mm
- net Net-(D50-Pad1): track 0.00 -> 13.1 mm
- net Net-(D26-Pad1): track 0.00 -> 13.0 mm
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Other:
- outline, holes or cut-outs redrawn
