File: PCB/CYOA_Ortho.kicad_sch (KiCad schematic)
At the start: 127 parts, among them U1 ProMicro

Commit message: routing pretty much done
Parts:
- added SW1: RotaryEncoder_Switch, Keebio-Parts:RotaryEncoder_EC11, symbol Device:RotaryEncoder_Switch
Connections:
- net GND: now also SW1.C
- net col1: now also U1.19 (A2/PF5); no longer U1.6 (3/PD0)
- net col2: now also U1.18 (A1/PF6); no longer U1.7 (4/PD4)
- net col3: now also U1.17 (A0/PF7); no longer U1.8 (5/PC6)
- net col4: now also U1.16 (15/PB1); no longer U1.9 (6/PD7)
- net col5: now also U1.15 (14/PB3); no longer U1.10 (7/PE6)
- net col6: now also U1.14 (16/PB2); no longer U1.11 (8/PB4)
- net col7: now also U1.13 (10/PB6); no longer U1.12 (9/PB5)
- net rowA: now also U1.5 (2/PD1); no longer U1.20 (A3/PF4)
- net rowB: now also U1.6 (3/PD0); no longer U1.19 (A2/PF5)
- net rowC: now also U1.7 (4/PD4); no longer U1.18 (A1/PF6)
- net rowD: now also U1.8 (5/PC6); no longer U1.17 (A0/PF7)
- net rowE: now also U1.9 (6/PD7); no longer U1.16 (15/PB1)
- net rowF: now also U1.10 (7/PE6); no longer U1.15 (14/PB3)
- net rowG: now also U1.11 (8/PB4); no longer U1.14 (16/PB2)
- net rowH: now also U1.12 (9/PB5); no longer U1.13 (10/PB6)
- net encA: now reaches U1.1 (TX0/PD3)
- net encA: now also SW1.A
- net encB: now reaches U1.2 (RX1/PD2)
- net encB: now also SW1.B
- net RotA: now reaches D1.1 (K), SW_A1.2
- net RotA: now also SW1.S1
- net col0 renamed RotB
- net RotB: now also U1.20 (A3/PF4), SW1.S2; no longer U1.5 (2/PD1)
- no-connect marks 4 -> 2
Other:
- moved on the sheet: D1, D10, D11, D12, D13, D14, D15, D16, D17, D18, D19, D2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

Commit message: Silkscreen mostly done
Parts:
- added SW2, SW3, SW4, SW5, SW6: RotaryEncoder_Switch, Keebio-Parts:RotaryEncoder_EC11, symbol Device:RotaryEncoder_Switch
Connections:
- net GND: now also SW2.C, SW3.C, SW4.C, SW5.C, SW6.C
- net encA: now also SW2.A, SW3.A, SW4.A, SW5.A, SW6.A
- net encB: now also SW2.B, SW3.B, SW4.B, SW5.B, SW6.B
- net D12RotA: now reaches D37.1 (K), SW_D12.2
- net D12RotA: now also SW5.S2
- net D1RotA: now reaches D48.1 (K), SW_D1.2
- net D1RotA: now also SW2.S2
- net A12RotA: now reaches D12.1 (K), SW_A12.2
- net A12RotA: now also SW4.S2
- net E12RotA: now reaches D49.1 (K), SW_E12.2
- net E12RotA: now also SW6.S2
- net E1RotA: now reaches D50.1 (K), SW_E1.2
- net E1RotA: now also SW3.S2
- net RotA renamed A1RotA
- net A1RotA: now also SW1.S2; no longer SW1.S1
- net RotB renamed A1RotB
- net A1RotB: now also SW1.S1, SW2.S1, SW3.S1; no longer SW1.S2
- net col3 renamed A12RotB
- net A12RotB: now also SW4.S1
- net col7 renamed D12RotB
- net D12RotB: now also SW5.S1, SW6.S1

Commit message: Version 0.1 done and sent to fabrication
Parts:
- added SW7, SW8: RotaryEncoder_Switch, Keebio-Parts:RotaryEncoder_EC11, symbol Device:RotaryEncoder_Switch
Connections:
- net A12RotB: now also SW8.S1
- net A1RotB: now also SW7.S1
- net GND: now also SW7.C, SW8.C
- net encA: now also SW7.A, SW8.A
- net encB: now also SW7.B, SW8.B
- net C1RotA: now reaches D26.1 (K), SW_C1.2
- net C1RotA: now also SW7.S2
- net C12RotA: now reaches D25.1 (K), SW_C12.2
- net C12RotA: now also SW8.S2
Other:
- moved on the sheet: SW1, SW4

Commit message: Pro micro footprint fixed v0.2 done
Parts:
- U1: footprint Keebio Parts:ArduinoProMicro-Mini-USB -> Keebio-Parts:ArduinoProMicro
Changed lines of the file:
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@@
       (effects (font (size 1.524 1.524)))
     )
-    (property "Footprint" "Keebio Parts:ArduinoProMicro-Mini-USB" (at 314.96 157.48 90)
+    (property "Footprint" "Keebio-Parts:ArduinoProMicro" (at 314.96 157.48 90)
       (effects (font (size 1.524 1.524)) hide)
     )

Commit message: Update to Kicad v8 and enlarged centre hole of switch to support Choc v2 switches too (this is in v0.4)
Parts:
- SW_A1, SW_A10, SW_A11, SW_A12, SW_A2, SW_A3, SW_A4, SW_A5, SW_A6, SW_A7, SW_A8, SW_A9, SW_B1, SW_B10, SW_B11, SW_B12, SW_B2, SW_B3, SW_B4, SW_B5, SW_B6, SW_B7, SW_B8, SW_B9, SW_C1, SW_C10, SW_C11, SW_C12, SW_C2, SW_C3, SW_C4, SW_C5, SW_C6, SW_C7, SW_C8, SW_C9, SW_D1, SW_D10, SW_D11, SW_D12, SW_D2, SW_D3, SW_D4, SW_D5, SW_D6, SW_D7, SW_D8, SW_D9, SW_E1, SW_E10, SW_E11, SW_E12, SW_E2, SW_E3, SW_E4, SW_E5, SW_E6, SW_E7, SW_E8, SW_E9: footprint Keebio-Parts:MX-Alps-Choc-1U-NoLED -> Keebio-Parts:MX-Alps-Choc-v1_v2-1U-NoLED
- SW_Da5, SW_Da6, SW_Da7, SW_Ea5, SW_Ea6, SW_Ea7: footprint Keebio-Parts:MX-Alps-Choc-2U-StabFlip-NoLED -> Keebio-Parts:MX-Alps-Choc-v1_v2-2U-StabFlip-NoLED
